File: SCHEMATIC/v1/guac_v2.brd (EAGLE design)
At the start: 41 x 50 mm, 31 parts, among them X1 STEREOJACK

Commit message: guac with dcdc, smart idea?
Parts:
- added GND, VIN: WIREPAD3,17/1,3, wirepad:3,17/1,3
- added Q1: 12mhz, crystal:HC49UP
- added U$3: LOGO_10X10_SILK, logo:LOGO_10X10_SILK
- added U$9: MP1584EN_FRAMELESS, power_supply:MP1584EN_FRAMELESS
- C1, C2: value (none) -> 22n, 885012207094
- C10, C9: value (none) -> 100u, VE-101M1CTR-0605
- C11, C12: value (none) -> 47u, VE-470M1CTR-0505
- C3, C4, C5, C8: value (none) -> 1u, 08055C105K4T2A
- C6, C7: value (none) -> 27p
- R1, R2: value (none) -> 15
- R11, R9: value (none) -> 1k5
- R12: value (none) -> 1M
- R3, R4, R5, R6: value (none) -> 3k3
- R7, R8: value (none) -> 22
- moved C12 162.9 mm to (20.0, 45.5)
- moved C11 142.0 mm to (10.2, 33.8), turned to 270 degrees
- moved C8 128.7 mm to (13.4, 42.4), turned to 90 degrees
- moved C7 123.1 mm to (28.0, 38.2), turned to 90 degrees
- moved C10 118.3 mm to (10.4, 18.6), turned to 90 degrees
- moved C9 112.6 mm to (30.5, 18.7), turned to 90 degrees
- moved C6 107.7 mm to (28.0, 26.3), turned to 270 degrees
- moved C5 101.3 mm to (17.3, 26.1)
- moved C4 97.6 mm to (10.9, 27.4), turned to 180 degrees
- moved R11 91.8 mm to (25.8, 38.3), turned to 90 degrees
- moved C3 91.5 mm to (11.0, 25.2)
- moved R12 90.8 mm to (28.0, 32.6), turned to 90 degrees
- moved R9 84.4 mm to (7.23, 42.3), turned to 270 degrees
- moved C2 83.8 mm to (16.5, 20.4), turned to 90 degrees
- moved C1 81.9 mm to (24.3, 20.4), turned to 90 degrees
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Connections:
- removed net AGNDL: U$1.AGNDL
- removed net AGNDR: U$1.AGNDR
- removed net HOST: U$1.HOST
- removed net N$8: C12.+, R11.2, R9.2, U$1.PSEL, U$1.VDD
- removed net PGND: U$1.PGND
- removed net VCCL: U$1.VCCL
- removed net VCCP: U$1.VCCP
- removed net VCCR: U$1.VCCR
- removed net VCOM: U$1.VCOM
- removed net ZGND: U$1.ZGND
- new net N$10: C6.1, Q1.1, R12.1, U$1.XTI
- new net N$11: C2.1, R2.2
- new net N$12: C5.2, U$1.VCCP
- new net N$13: C1.2, C9.+, R3.2, U$1.VOUTL
- new net N$14: C11.+, U$1.VCOM
- new net N$15: C10.+, C2.2, R4.2, U$1.VOUTR
- new net N$16: C4.1, U$1.VCCR
- new net N$17: C9.-, R5.2, X1.5
- new net N$18: C1.1, R1.2
- new net N$19: C10.-, R6.2, X1.2
- new net N$20: C3.2, U$1.VCCL
- new net N$6: JP1.SHELL, U$1.DOUT
- new net N$9: C7.1, Q1.2, R12.2, U$1.XTO
- new net VCC: C12.+, R11.2, R9.2, U$1.FSEL, U$1.HOST, U$1.PSEL, U$1.TEST, U$1.VDD
- new net VIN: U$9.VIN, VIN.1
- net GND: now also C11.-, C3.1, C4.2, C5.1, C6.2, C7.2, GND.1, JP1.PIN, JP1.SWITCH, R1.1, R2.1, R3.1, R4.1, R5.1, R6.1, U$1.AGNDL, U$1.AGNDR, U$1.PGND, U$1.ZGND, U$9.GNDIN, U$9.GNDOUT, X1.1
- net VREG: now also U$9.VOUT
Routing:
- net GND: track 0.00 -> 257.7 mm, vias 0 -> 3
- net VCC: track 0.00 -> 68.6 mm, vias 0 -> 3
- net VIN: track 0.00 -> 55.6 mm, vias 0 -> 3
- net VREG: track 0.00 -> 53.6 mm
- net N$6: track 0.00 -> 42.6 mm, vias 0 -> 1
- net N$13: track 0.00 -> 35.9 mm, vias 0 -> 2
- net N$15: track 0.00 -> 26.5 mm, vias 0 -> 2
- net N$19: track 0.00 -> 23.6 mm
- net N$17: track 0.00 -> 18.5 mm
- net N$1: track 0.00 -> 16.0 mm, vias 0 -> 2
- net N$20: track 0.00 -> 14.6 mm, vias 0 -> 2
- net N$2: track 0.00 -> 13.7 mm
- net N$10: track 0.00 -> 12.3 mm
- net N$4: track 0.00 -> 11.9 mm
- net N$9: track 0.00 -> 10.7 mm
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Other:
- board text added: "GUAC DIP"
- board text added: "JKW v0.1"
- board text removed: "JKW v3.b"
- board text removed: "JKW v3.c"
- board text removed: "SALSA DIP II"
